File: SR_Testing_Rig_Schematics/SR_Testing_Rig_Schematics.kicad_sch (KiCad schematic)
At the start: 5 parts, among them Q1_Power NPN, U1 ESP32-WROOM-32, U2 LT1963AxST-3.3

Commit message: schematic update
Other:
- note added: "Linear regulator"
- moved on the sheet: A1, Q1_Power, R_batt, U1, U2
